Commit message: claw and rod,but pid not ready

File: resources/robots/claw2/urdf/claw4.urdf (robot description, URDF)
Before this commit: robot claw4, 5 links, 4 joints
Joints:
- joint P_1_to_2_Link: limit lower=-3.14 upper=3.14 effort=300 velocity=100 -> lower=-3.14 upper=3.14 effort=200000000000000000 velocity=100
- joint P_2_to_left_Link: limit lower=-3.14 upper=3.14 effort=300 velocity=100 -> lower=-3.14 upper=3.14 effort=20000000000000000 velocity=100
- joint P_2_to_right_Link: limit lower=-3.14 upper=3.14 effort=300 velocity=100 -> lower=-3.14 upper=3.14 effort=20000000000 velocity=100
- joint P_base_to_1_Link: limit lower=-3.14 upper=3.14 effort=300 velocity=100 -> lower=-3.14 upper=3.14 effort=20000000000000000000 velocity=100

File: resources/robots/claw4/urdf/claw4.urdf (robot description, URDF)
Before this commit: robot claw4.SLDASM, 5 links, 4 joints
Links:
- link P_1_Link: geometry collision mesh filename=../meshes/P_1_Link.STL; visual mesh filename=../meshes/P_1_Link.STL
- link P_2_Link: geometry collision mesh filename=../meshes/P_2_Link.STL; visual mesh filename=../meshes/P_2_Link.STL
- link P_base_Link: geometry collision mesh filename=../meshes/P_base_Link.STL; visual mesh filename=../meshes/P_base_Link.STL
- link P_left_Link: geometry collision mesh filename=../meshes/P_left_Link.STL; visual mesh filename=../meshes/P_left_Link.STL
- link P_right_Link: geometry collision mesh filename=../meshes/P_right_Link.STL; visual mesh filename=../meshes/P_right_Link.STL
Joints:
- joint P_2_to_left_Link: limit lower=-3.14 upper=3.14 effort=300 velocity=100 -> lower=-3.14 upper=3.14 effort=10000 velocity=100
- joint P_2_to_right_Link: limit lower=-3.14 upper=3.14 effort=300 velocity=100 -> lower=-3.14 upper=3.14 effort=10000 velocity=100
- joint P_base_to_1_Link: limit lower=-3.14 upper=3.14 effort=300 velocity=100 -> lower=-3.14 upper=3.14 effort=10000 velocity=100
