Commit message: pid retune

File: resources/robots/claw4/urdf/claw4.urdf (robot description, URDF)
Before this commit: robot claw4, 5 links, 4 joints
Joints:
- joint P_1_to_2_Link: limit lower=-3.14 upper=3.14 effort=300 velocity=100 -> lower=-3.14 upper=3.14 effort=200 velocity=100
- joint P_2_to_left_Link: limit lower=-3.14 upper=3.14 effort=10000 velocity=100 -> lower=-3.14 upper=3.14 effort=120 velocity=100
- joint P_2_to_right_Link: limit lower=-3.14 upper=3.14 effort=10000 velocity=100 -> lower=-3.14 upper=3.14 effort=120 velocity=100
- joint P_base_to_1_Link: limit lower=-3.14 upper=3.14 effort=10000 velocity=100 -> lower=-3.14 upper=3.14 effort=200 velocity=100
