Commit message: can train

File: resources/robots/claw4(original)/urdf/claw4.urdf (robot description, URDF)
Before this commit: robot claw and rod, 5 links, 4 joints
Links:
- link P_1_Link: mass 2.29977871437821 -> 2.2998
- link P_2_Link: mass 6.27444678594554 -> 6.2744
- link P_base_Link: mass 6.45985390928753 -> 6.4599
- link P_left_Link: mass 2.8207521601036 -> 2.8208
- link P_right_Link: mass 2.8207521601036 -> 2.8208
Joints:
- joint P_1_to_2_Link: limit lower=-3.14 upper=3.14 effort=2000000000000000000 velocity=20 -> lower=-3.14 upper=3.14 effort=400 velocity=100; origin xyz=-0.125 -0.00079057 0 rpy=1.5708 0.18691 -3.1353 -> xyz=-0.12499 -0.0011962 0 rpy=1.5708 0.17993 -3.132
- joint P_2_to_left_Link: limit lower=-3.14 upper=3.14 effort=50000000000000000000000 velocity=20 -> lower=-3.14 upper=3.14 effort=120 velocity=100; origin xyz=0.30414 0 0 rpy=3.1416 0 -1.4056 -> xyz=0.30414 0 0 rpy=-3.1416 0 -1.4056
- joint P_2_to_right_Link: limit lower=-3.14 upper=3.14 effort=50000000000000000000 velocity=20 -> lower=-3.14 upper=3.14 effort=120 velocity=100
- joint P_base_to_1_Link: limit lower=-3.14 upper=3.14 effort=200000000000000000000000000 velocity=20 -> lower=-3.14 upper=3.14 effort=200 velocity=100; origin xyz=-0.011518 0 -0.36982 rpy=-1.5708 -1.5397 0 -> xyz=0 0 -0.37 rpy=1.5708 -1.5708 0

File: resources/robots/claw4(test)/urdf/claw4.urdf (robot description, URDF)
Before this commit: robot claw and rod, 5 links, 4 joints
Joints:
- joint P_1_to_2_Link: child P_2_Link -> P_1_Link; limit lower=-3.14 upper=3.14 effort=2000000000000000000 velocity=20 -> lower=-3.14 upper=3.14 effort=200 velocity=20; origin xyz=-0.125 -0.00079057 0 rpy=1.5708 0.18691 -3.1353 -> xyz=-0.05 0.3 0 rpy=-3.1416 0 -1.4056; parent P_1_Link -> P_2_Link
- joint P_2_to_left_Link: child P_left_Link -> P_2_Link; limit lower=-3.14 upper=3.14 effort=50000000000000000000000 velocity=20 -> lower=-3.14 upper=3.14 effort=200 velocity=20; origin xyz=0.30414 0 0 rpy=3.1416 0 -1.4056 -> xyz=0 0 0 rpy=0 0 0; parent P_2_Link -> P_left_Link
- joint P_2_to_right_Link: limit lower=-3.14 upper=3.14 effort=50000000000000000000 velocity=20 -> lower=-3.14 upper=3.14 effort=200 velocity=20; origin xyz=0.2877 0.098639 0 rpy=0 0 -1.4056 -> xyz=-0.1 0 0 rpy=3.1416 0 0
- joint P_base_to_1_Link: child P_1_Link -> P_base_Link; limit lower=-3.14 upper=3.14 effort=200000000000000000000000000 velocity=20 -> lower=-3.14 upper=3.14 effort=200 velocity=20; origin xyz=-0.011518 0 -0.36982 rpy=-1.5708 -1.5397 0 -> xyz=-0.12282 -0.023228 0 rpy=1.5708 0.0063246 -2.9547; parent P_base_Link -> P_1_Link
