Commit message: 2dofs version

File: resources/obj/rod/urdf/rod.urdf (robot description, URDF)
Before this commit: robot rod, 1 links, 0 joints
Links:
- link rod_Link: geometry collision cylinder length=0.8 radius=0.04; visual cylinder length=0.8 radius=0.04

File: resources/robots/claw4/urdf/claw4.urdf (robot description, URDF)
Before this commit: robot claw and rod, 5 links, 4 joints
Joints:
- joint P_1_to_2_Link: limit lower=-3.14 upper=3.14 effort=2000000000000000000 velocity=20 -> lower=-3.14 upper=3.14 effort=100 velocity=20
- joint P_2_to_left_Link: origin xyz=0.30414 0 0 rpy=3.1416 0 -1.4056 -> xyz=0.30414 0 0 rpy=3.1416 0 -1.22; type revolute -> fixed
- joint P_2_to_right_Link: origin xyz=0.2877 0.098639 0 rpy=0 0 -1.4056 -> xyz=0.2877 0.098639 0 rpy=0 0 -1.78; type revolute -> fixed
- joint P_base_to_1_Link: limit lower=-3.14 upper=3.14 effort=200000000000000000000000000 velocity=20 -> lower=-3.14 upper=3.14 effort=100  velocity=20

Commit message: 2dofs cant balance but can stand up through big friction

File: resources/obj/rod/urdf/rod.urdf (robot description, URDF)
Before this commit: robot rod, 1 links, 0 joints
Links:
- link rod_Link: geometry collision cylinder length=0.8 radius=0.039; visual cylinder length=0.8 radius=0.039

File: resources/robots/claw4(方形）/urdf/claw4.urdf (robot description, URDF)
Before this commit: robot claw4, 5 links, 4 joints
Links:
- link P_2_Link: mass 6.27444678594553 -> 6.27444678594554
- link P_left_Link: mass 3.6405391689699 -> 2.8207521601036
- link P_right_Link: mass 3.6405391689699 -> 2.8207521601036
Joints:
- joint P_1_to_2_Link: limit lower=-3.14 upper=3.14 effort=100 velocity=10 -> lower=-3.14 upper=3.14 effort=100 velocity=20; origin xyz=-0.124982724435145 0.00207812241333377 0 rpy=1.5707963267949 1.38898656478725 3.12496690835837 -> xyz=-0.125 -0.00079057 0 rpy=1.5708 0.18691 -3.1353
- joint P_2_to_left_Link: axis -0.28312 0.0047175 0.95907 -> 0 0 -1; limit lower=-3.14 upper=3.14 effort=500000000 velocity=10 -> lower=-3.14 upper=3.14 effort=50000000000000000000000 velocity=20; origin xyz=0 0.30414 0 rpy=0 0 -1.7359 -> xyz=0.30414 0 0 rpy=3.1416 0 -1.22
- joint P_2_to_right_Link: axis -0.281861633691698 -0.0270656193743369 0.959073235837874 -> 0 0 -1; limit lower=-3.14 upper=3.14 effort=500000000 velocity=10 -> lower=-3.14 upper=3.14 effort=50000000000000000000 velocity=20; origin xyz=0.0986393923832151 0.287698227784404 0 rpy=3.14159265358979 0 1.48471753829469 -> xyz=0.2877 0.098639 0 rpy=0 0 -1.78
- joint P_base_to_1_Link: limit lower=-3.14 upper=3.14 effort=100 velocity=10 -> lower=-3.14 upper=3.14 effort=100  velocity=20; origin xyz=-0.0115182488057926 0 -0.369820672684002 rpy=-1.57079632679488 -1.53966089433424 0 -> xyz=-0.011518 0 -0.36982 rpy=-1.5708 -1.5397 0

Commit message: success

File: resources/obj/rod/urdf/rod.urdf (robot description, URDF)
Before this commit: robot rod, 1 links, 0 joints
Links:
- link rod_Link: geometry collision cylinder length=0.8 radius=0.041; visual cylinder length=0.8 radius=0.041

File: resources/robots/claw4(分解不出来的尖v槽）/urdf/claw4.urdf (robot description, URDF)
Before this commit: robot claw4, 5 links, 4 joints
Links:
- link P_left_Link: mass 3.42978569666941 -> 4.58036974856787
- link P_right_Link: mass 3.42978569666941 -> 4.58036974856787
Joints:
- joint P_1_to_2_Link: origin xyz=-0.125 0.00079745 0 rpy=1.5708 1.4048 3.1352 -> xyz=-0.124997456248677 0.000797453039112106 0 rpy=1.57079632679489 1.39170475447566 3.13521298600109
- joint P_2_to_left_Link: axis -0.27332 0.00021897 0.96192 -> -0.273290136443592 0.00381070259111247 0.961924102966759; origin xyz=0 0.30414 0 rpy=0 0 -1.7359 -> xyz=0 0.304138126515083 0 rpy=0 0 -1.73594500421685; type revolute -> continuous
- joint P_2_to_right_Link: axis -0.27288 -0.015359 0.96192 -> -0.272884794791439 -0.015359326262194 0.96192410296676; origin xyz=0.098639 0.2877 0 rpy=-3.1416 0 1.4611 -> xyz=0.0986393923834267 0.287698227783769 0 rpy=-3.14159265358979 0 1.447930450626; type revolute -> continuous
- joint P_base_to_1_Link: origin xyz=-0.011518 0 -0.36982 rpy=-1.5708 -1.5397 0 -> xyz=-0.0115182488057926 0 -0.369820672684002 rpy=-1.57079632679488 -1.53966089433424 0

File: resources/robots/claw4(同样分解不出来）/urdf/claw4.urdf (robot description, URDF)
Before this commit: robot claw4, 5 links, 4 joints
Links:
- link P_left_Link: mass 3.42978569666941 -> 3.97303178078042
- link P_right_Link: mass 3.42978569666941 -> 3.97303178078042
Joints:
- joint P_1_to_2_Link: origin xyz=-0.125 0.00079745 0 rpy=1.5708 1.4048 3.1352 -> xyz=-0.12499745623252 0.000797453040616403 0 rpy=1.57079632679489 1.40484650611732 3.13521298600109
- joint P_2_to_left_Link: axis -0.27332 0.00021897 0.96192 -> -0.27331661527534 0.000218965812425212 0.961924102966759; origin xyz=0 0.30414 0 rpy=0 0 -1.7359 -> xyz=0 0.304138126533306 0 rpy=0 0 -1.73594500420734
- joint P_2_to_right_Link: axis -0.27288 -0.015359 0.96192 -> -0.272884794791439 -0.015359326262194 0.96192410296676; origin xyz=0.098639 0.2877 0 rpy=-3.1416 0 1.4611 -> xyz=0.098639392383322 0.287698227802974 0 rpy=-3.14159265358979 0 1.46107220226766
- joint P_base_to_1_Link: origin xyz=-0.011518 0 -0.36982 rpy=-1.5708 -1.5397 0 -> xyz=-0.0115182488057926 0 -0.369820672684002 rpy=-1.57079632679488 -1.53966089433424 0

File: resources/robots/claw4(方形被损坏）/urdf/claw4.urdf (robot description, URDF)
Before this commit: robot claw4, 5 links, 4 joints
Links:
- link P_1_Link: mass 2.29977871437822 -> 2.29977871437821
- link P_2_Link: mass 6.27444678594553 -> 6.27444678594554
- link P_left_Link: mass 3.42978569666941 -> 2.8207521601036
- link P_right_Link: mass 3.42978569666941 -> 2.8207521601036
Joints:
- joint P_1_to_2_Link: limit lower=-3.14 upper=3.14 effort=100 velocity=10 -> lower=-3.14 upper=3.14 effort=2000000000000000000 velocity=20; origin xyz=-0.125 0.00079745 0 rpy=1.5708 1.4048 3.1352 -> xyz=-0.125 -0.00079057 0 rpy=1.5708 0.18691 -3.1353
- joint P_2_to_left_Link: axis -0.27332 0.00021897 0.96192 -> 0 0 -1; limit lower=-3.14 upper=3.14 effort=500000000 velocity=10 -> lower=-3.14 upper=3.14 effort=50000000000000000000000 velocity=20; origin xyz=0 0.30414 0 rpy=0 0 -1.7359 -> xyz=0.30414 0 0 rpy=3.1416 0 -1.4056
- joint P_2_to_right_Link: axis -0.27288 -0.015359 0.96192 -> 0 0 -1; limit lower=-3.14 upper=3.14 effort=500000000 velocity=10 -> lower=-3.14 upper=3.14 effort=50000000000000000000 velocity=20; origin xyz=0.098639 0.2877 0 rpy=-3.1416 0 1.4611 -> xyz=0.2877 0.098639 0 rpy=0 0 -1.4056
- joint P_base_to_1_Link: limit lower=-3.14 upper=3.14 effort=100 velocity=10 -> lower=-3.14 upper=3.14 effort=200000000000000000000000000 velocity=20

File: resources/robots/claw4(环形）/urdf/claw4.urdf (robot description, URDF)
Before this commit: robot claw4, 5 links, 4 joints
Links:
- link P_1_Link: mass 2.29977871437822 -> 2.29977871437821
- link P_left_Link: mass 3.42978569666941 -> 3.6405391689699
- link P_right_Link: mass 3.42978569666941 -> 3.6405391689699
Joints:
- joint P_1_to_2_Link: origin xyz=-0.125 0.00079745 0 rpy=1.5708 1.4048 3.1352 -> xyz=-0.124982724435145 0.00207812241333377 0 rpy=1.5707963267949 1.38898656478725 3.12496690835837
- joint P_2_to_left_Link: axis -0.27332 0.00021897 0.96192 -> -0.28312 0.0047175 0.95907
- joint P_2_to_right_Link: axis -0.27288 -0.015359 0.96192 -> -0.281861633691698 -0.0270656193743369 0.959073235837874; origin xyz=0.098639 0.2877 0 rpy=-3.1416 0 1.4611 -> xyz=0.0986393923832151 0.287698227784404 0 rpy=3.14159265358979 0 1.48471753829469
- joint P_base_to_1_Link: origin xyz=-0.011518 0 -0.36982 rpy=-1.5708 -1.5397 0 -> xyz=-0.0115182488057926 0 -0.369820672684002 rpy=-1.57079632679488 -1.53966089433424 0
