Commit message: initial graduation project code

File: resources/obj/rod/urdf/15.urdf (robot description, URDF)
Before this commit: robot rod, 1 links, 0 joints
Links:
- link rod_Link: geometry collision cylinder length=0.8 radius=0.015; visual cylinder length=0.8 radius=0.015

File: resources/obj/rod/urdf/18.urdf (robot description, URDF)
Before this commit: robot rod, 1 links, 0 joints
Links:
- link rod_Link: geometry collision cylinder length=0.8 radius=0.018; visual cylinder length=0.8 radius=0.018

File: resources/obj/rod/urdf/20.urdf (robot description, URDF)
Before this commit: robot rod, 1 links, 0 joints
Links:
- link rod_Link: geometry collision cylinder length=0.8 radius=0.020; visual cylinder length=0.8 radius=0.020

File: resources/obj/rod/urdf/23.urdf (robot description, URDF)
Before this commit: robot rod, 1 links, 0 joints
Links:
- link rod_Link: geometry collision cylinder length=0.8 radius=0.023; visual cylinder length=0.8 radius=0.023

File: resources/obj/rod/urdf/25.urdf (robot description, URDF)
Before this commit: robot rod, 1 links, 0 joints
Links:
- link rod_Link: geometry collision cylinder length=0.8 radius=0.025; visual cylinder length=0.8 radius=0.025

File: resources/obj/rod/urdf/27.urdf (robot description, URDF)
Before this commit: robot rod, 1 links, 0 joints
Links:
- link rod_Link: geometry collision cylinder length=0.8 radius=0.027; visual cylinder length=0.8 radius=0.027

File: resources/obj/rod/urdf/30.urdf (robot description, URDF)
Before this commit: robot rod, 1 links, 0 joints
Links:
- link rod_Link: geometry collision cylinder length=0.8 radius=0.030; visual cylinder length=0.8 radius=0.030

File: resources/obj/rod/urdf/32.urdf (robot description, URDF)
Before this commit: robot rod, 1 links, 0 joints
Links:
- link rod_Link: geometry collision cylinder length=0.8 radius=0.032; visual cylinder length=0.8 radius=0.032

File: resources/obj/rod/urdf/37.urdf (robot description, URDF)
Before this commit: robot rod, 1 links, 0 joints
Links:
- link rod_Link: geometry collision cylinder length=0.8 radius=0.037; visual cylinder length=0.8 radius=0.037

File: resources/obj/rod/urdf/39.urdf (robot description, URDF)
Before this commit: robot rod, 1 links, 0 joints
Links:
- link rod_Link: geometry collision cylinder length=0.8 radius=0.039; visual cylinder length=0.8 radius=0.039

File: resources/robots/claw4/urdf/claw4.urdf (robot description, URDF)
Before this commit: robot claw4, 5 links, 4 joints
Joints:
- joint P_1_to_2_Link: limit lower=-3.14 upper=3.14 effort=100 velocity=10 -> lower=-3.14 upper=3.14 effort=150 velocity=10
- joint P_base_to_1_Link: limit lower=-3.14 upper=3.14 effort=100 velocity=10 -> lower=-3.14 upper=3.14 effort=150 velocity=10
